File: hardware/kicad/can-node-breakout/can-node-breakout.kicad_pcb (KiCad board)
At the start: 2 copper layers, 45.5 x 25 mm, 48 parts, among them J1 Conn_01x04_Male, J12 Conn_01x04_Male, J13 Conn_01x02_Male, J21 Conn_01x06_Male, J22 Conn_01x06_Male, J23 Conn_01x04_Male, SW21 SW_Push, U1 ADM3053, U12 TPS73233_SOT23_5, U22 STM32F042K6Tx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

Commit message: Added rev. 2.
Parts:
- moved C7 0.38 mm to (93.7, 121.2)
- moved C8 0.38 mm to (93.7, 119.6)
Routing:
- net (no net): track 122.7 -> 18.5 mm, vias 1 -> 0
- net /can_interface/3V3: track 119.4 -> 124.8 mm, vias 19 -> 20
Other:
- net class Default: clearance 0.2 -> 0.1
- rule trace_clearance: 0.2 -> 0.1
Changed lines of the file:
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@@
     (thickness 1.6)
     (drawings 7)
-    (tracks 519)
+    (tracks 497)
     (zones 0)
     (modules 48)
@@
   (setup
     (last_trace_width 0.25)
-    (trace_clearance 0.2)
-    (zone_clearance 0.508)
+    (trace_clearance 0.1)
+    (zone_clearance 0.2)
     (zone_45_only no)
     (trace_min 0.2)
@@
   (net 47 "Net-(U22-Pad6)")
   (net_class Default "This is the default net class."
-    (clearance 0.2)
+    (clearance 0.1)
     (trace_width 0.25)
     (via_dia 0.8)
@@
     (add_net "Net-(U22-Pad9)")
   )
+  (module Mounting_Holes:MountingHole_2.2mm_M2 (layer F.Cu)
+    (at 92.456 107.442)
+    (descr "Mounting Hole 2.2mm, no annular, M2")
+    (tags "mounting hole 2.2mm no annular m2")
+    (attr virtual)
+    (fp_text reference H1 (at 0 -3.2) (layer F.SilkS) hide
+      (effects (font (size 1 1) (thickness 0.15)))
+    )
+    (fp_text value MountingHole (at 0 3.2) (layer F.Fab) hide
+      (effects (font (size 1 1) (thickness 0.15)))
+    )
+    (fp_circle (center 0 0) (end 2.45 0) (layer F.CrtYd) (width 0.05))
+    (fp_circle (center 0 0) (end 2.2 0) (layer Cmts.User) (width 0.15))
+    (fp_text user %R (at 0.3 0) (layer F.Fab) hide
+      (effects (font (size 1 1) (thickness 0.15)))
+    )
+    (pad 1 np_thru_hole circle (at 0 0) (size 2.2 2.2) (drill 2.2) (layers *.Cu *.Mask))
+  )
   (module Capacitors_SMD:C_0603 (layer F.Cu)
     (at 111.76 123.19 180)
@@
   )
   (module Capacitors_SMD:C_0603 (layer F.Cu)
-    (at 93.651911 121.534668 180)
+    (at 93.651911 121.158 180)
     (descr "Capacitor SMD 0603, reflow soldering, AVX (see smccp.pdf)")
     (tags "capacitor 0603")
@@
   )
   (module Capacitors_SMD:C_0603 (layer F.Cu)
-    (at 93.651911 120.010668 180)
+    (at 93.651911 119.634 180)
     (descr "Capacitor SMD 0603, reflow soldering, AVX (see smccp.pdf)")
     (tags "capacitor 0603")
@@
   )
   (module Mounting_Holes:MountingHole_2.2mm_M2 (layer F.Cu)
-    (at 92.456 107.442)
-    (descr "Mounting Hole 2.2mm, no annular, M2")
-    (tags "mounting hole 2.2mm no annular m2")
-    (attr virtual)
-    (fp_text reference H1 (at 0 -3.2) (layer F.SilkS) hide
-      (effects (font (size 1 1) (thickness 0.15)))
-    )
-    (fp_text value MountingHole (at 0 3.2) (layer F.Fab) hide
-      (effects (font (size 1 1) (thickness 0.15)))
-    )
-    (fp_circle (center 0 0) (end 2.45 0) (layer F.CrtYd) (width 0.05))
-    (fp_circle (center 0 0) (end 2.2 0) (layer Cmts.User) (width 0.15))
-    (fp_text user %R (at 0.3 0) (layer F.Fab) hide
-      (effects (font (size 1 1) (thickness 0.15)))
-    )
-    (pad 1 np_thru_hole circle (at 0 0) (size 2.2 2.2) (drill 2.2) (layers *.Cu *.Mask))
-  )
-  (module Mounting_Holes:MountingHole_2.2mm_M2 (layer F.Cu)
     (at 92.456 127.254)
     (descr "Mounting Hole 2.2mm, no annular, M2")
@@
   (gr_line (start 135.5 105) (end 135.5 130) (layer Edge.Cuts) (width 0.15))
   (gr_line (start 90 105) (end 135.5 105) (layer Edge.Cuts) (width 0.15))
-  (segment (start 112.369 106.2) (end 108.619 106.2) (width 0.25) (layer F.Cu) (net 0))
-  (segment (start 112.869 106.2) (end 112.369 106.2) (width 0.25) (layer F.Cu) (net 0))
-  (segment (start 103.434 106.604) (end 96.984 106.604) (width 0.25) (layer F.Cu) (net 0))
-  (segment (start 104.184 106.604) (end 103.434 106.604) (width 0.25) (layer F.Cu) (net 0))
-  (segment (start 97.734 128.092) (end 104.184 128.092) (width 0.25) (layer F.Cu) (net 0))
-  (segment (start 96.984 128.092) (end 97.734 128.092) (width 0.25) (layer F.Cu) (net 0))
-  (via (at 96.984 106.604) (size 0.8) (drill 0.4) (layers F.Cu B.Cu) (net 0))
-  (segment (start 93.294 106.604) (end 92.456 107.442) (width 0.25) (layer F.Cu) (net 0))
-  (segment (start 96.984 106.604) (end 93.294 106.604) (width 0.25) (layer F.Cu) (net 0))
-  (segment (start 91.356001 126.154001) (end 92.456 127.254) (width 0.25) (layer B.Cu) (net 0))
   (segment (start 90.772999 125.570999) (end 91.356001 126.154001) (width 0.25) (layer B.Cu) (net 0))
   (segment (start 90.772999 109.125001) (end 90.772999 125.570999) (width 0.25) (layer B.Cu) (net 0))
-  (segment (start 92.456 107.442) (end 90.772999 109.125001) (width 0.25) (layer B.Cu) (net 0))
   (segment (start 93.294 128.092) (end 92.456 127.254) (width 0.25) (layer F.Cu) (net 0))
-  (segment (start 96.984 128.092) (end 93.294 128.092) (width 0.25) (layer F.Cu) (net 0))
-  (segment (start 131.742001 106.342001) (end 132.842 107.442) (width 0.25) (layer F.Cu) (net 0))
-  (segment (start 130.86799 105.46799) (end 131.742001 106.342001) (width 0.25) (layer F.Cu) (net 0))
-  (segment (start 114.10101 105.46799) (end 130.86799 105.46799) (width 0.25) (layer F.Cu) (net 0))
-  (segment (start 113.369 106.2) (end 114.10101 105.46799) (width 0.25) (layer F.Cu) (net 0))
-  (segment (start 112.869 106.2) (end 113.369 106.2) (width 0.25) (layer F.Cu) (net 0))
-  (segment (start 133.941999 126.408001) (end 132.842 127.508) (width 0.25) (layer B.Cu) (net 0))
-  (segment (start 135.09999 125.25001) (end 133.941999 126.408001) (width 0.25) (layer B.Cu) (net 0))
-  (segment (start 135.09999 109.69999) (end 135.09999 125.25001) (width 0.25) (layer B.Cu) (net 0))
-  (segment (start 132.842 107.442) (end 135.09999 109.69999) (width 0.25) (layer B.Cu) (net 0))
-  (segment (start 104.934 128.092) (end 104.184 128.092) (width 0.25) (layer F.Cu) (net 0))
-  (segment (start 106.345001 129.503001) (end 104.934 128.092) (width 0.25) (layer F.Cu) (net 0))
-  (segment (start 130.846999 129.503001) (end 106.345001 129.503001) (width 0.25) (layer F.Cu) (net 0))
-  (segment (start 132.842 127.508) (end 130.846999 129.503001) (width 0.25) (layer F.Cu) (net 0))
   (via (at 128.27 124.206) (size 0.8) (drill 0.4) (layers F.Cu B.Cu) (net 1))
   (segment (start 106.045 111.973) (end 106.045 112.648) (width 0.25) (layer F.Cu) (net 1))
@@
   (segment (start 130.932347 128.392347) (end 130.932347 124.591653) (width 0.25) (layer B.Cu) (net 3))
   (segment (start 130.932347 124.591653) (end 131.826 123.698) (width 0.25) (layer B.Cu) (net 3))
+  (via (at 130.048 121.412) (size 0.8) (drill 0.4) (layers F.Cu B.Cu) (net 3))
+  (segment (start 130.048 118.872) (end 128.016 116.84) (width 0.25) (layer B.Cu) (net 3))
+  (segment (start 130.048 121.412) (end 130.048 118.872) (width 0.25) (layer B.Cu) (net 3))
   (segment (start 98.709 125.492) (end 98.709 124.892) (width 0.25) (layer F.Cu) (net 4))
   (segment (start 104.694003 126.117001) (end 99.334001 126.117001) (width 0.25) (layer F.Cu) (net 4))
@@
     )
   )
+  (zone (net 2) (net_name "Net-(C1-Pad1)") (layer F.Cu) (hatch full 0.508)
+    (priority 3)
+    (connect_pads yes (clearance 0.2))
+    (min_thickness 0.2)
+    (fill yes (arc_segments 32) (thermal_gap 0.508) (thermal_bridge_width 0.508))
+    (polygon
+      (pts
+        (xy 106.172 127.762) (xy 109.474 127.762) (xy 109.474 126.492) (xy 113.284 126.492) (xy 113.284 124.46)
+        (xy 111.76 124.46) (xy 111.76 125.984) (xy 110.744 125.984) (xy 110.744 124.46) (xy 109.728 124.46)
+        (xy 108.204 125.984) (xy 106.172 125.984)
+      )
+    )
+  )
+  (zone (net 3) (net_name /can_interface/3V3) (layer F.Cu) (hatch full 0.508)
+    (priority 2)
+    (connect_pads yes (clearance 0.508))
+    (min_thickness 0.254)
+    (fill yes (arc_segments 16) (thermal_gap 0.508) (thermal_bridge_width 0.508))
+    (polygon
+      (pts
+        (xy 93.98 121.666) (xy 96.266 121.666) (xy 96.266 118.364) (xy 93.98 118.364)
+      )
+    )
+  )
+  (zone (net 3) (net_name /can_interface/3V3) (layer F.Cu) (hatch full 0.508)
+    (priority 2)
+    (connect_pads yes (clearance 0.508))
+    (min_thickness 0.254)
+    (fill yes (arc_segments 16) (thermal_gap 0.508) (thermal_bridge_width 0.508))
+    (polygon
+      (pts
+        (xy 129.286 125.476) (xy 132.588 125.476) (xy 132.588 122.428) (xy 131.064 122.428) (xy 131.064 120.904)
+        (xy 129.286 120.904)
+      )
+    )
+  )
   (zone (net 1) (net_name GND) (layer F.Cu) (hatch full 0.508)
     (priority 1)
@@
     (polygon
       (pts
-        (xy 89.408 104.394) (xy 135.636 104.394) (xy 135.636 131.064) (xy 89.154 131.064)
+        (xy 89.408 104.14) (xy 136.144 103.886) (xy 136.144 132.842) (xy 88.9 132.334)
       )
     )
@@
     (polygon
       (pts
-        (xy 89.420814 104.394) (xy 135.648814 104.394) (xy 135.648814 131.064) (xy 89.166814 131.064)
+        (xy 89.408 104.14) (xy 136.144 103.886) (xy 136.144 132.842) (xy 88.9 132.334)
       )
     )
-  )
-  (zone (net 2) (net_name "Net-(C1-Pad1)") (layer F.Cu) (hatch full 0.508)
-    (priority 2)
-    (connect_pads yes (clearance 0.508))
-    (min_thickness 0.254)
-    (fill yes (arc_segments 16) (thermal_gap 0.508) (thermal_bridge_width 0.508))
-    (polygon
-      (pts
-        (xy 106.172 127.762) (xy 109.474 127.762) (xy 109.474 126.492) (xy 113.284 126.492) (xy 113.284 124.46)
-        (xy 111.76 124.46) (xy 111.76 125.984) (xy 110.744 125.984) (xy 110.744 124.46) (xy 109.728 124.46)
-        (xy 108.204 125.984) (xy 106.172 125.984)
-      )
-    )
-  )
-  (zone (net 3) (net_name /can_interface/3V3) (layer F.Cu) (hatch full 0.508)
-    (priority 1)
-    (connect_pads yes (clearance 0.508))
-    (min_thickness 0.254)
-    (fill yes (arc_segments 16) (thermal_gap 0.508) (thermal_bridge_width 0.508))
-    (polygon
-      (pts
-        (xy 87.122 101.854) (xy 138.684 101.854) (xy 138.43 133.604) (xy 87.376 134.366)
-      )
-    )
